File: eagle/marionette.sch (EAGLE design)
At the start: 58 parts, among them J2 SWD_CONNECTOR, J3 2X10FE, J4 2X10FE, J5 2X10FE, J6 2X10FE, J7 2X10FE, U1 USB3318, U2 NCP705, U3 XCL206B, X1 ABS25-32.768KHZ-6-T

Commit message: Added connections to the EDGE CONNECTOR OF DEATH!!!!!!!!!!!!!
Parts:
- added C31: 100nF, 10V, rcl_custom:C-EU0603-C
- added U$15: PTS645, PTS645:PTS645
- C27: device rcl_custom:C-EU0603-C -> rcl_custom:C-EU0402-C
Connections:
- new net I2C2_SCL: R3.1, U$1G$6.PF1
- new net I2C2_SLC: J3.19
- new net N$13: C31.1, U$15.P$2, U$1G$11.NRST
- net ADC1/2/3_IN11: now also J7.4
- net ADC1/2/3_IN13: now also J7.5
- net ADC1/2/3_IN2: now also J7.1
- net ADC1/2_IN14: now also J7.6
- net ADC1/2_IN15: now also J7.7
- net ADC1/2_IN6: now also J7.2
- net ADC1/2_IN7: now also J7.3
- net ADC3_IN14: now also J7.9
- net ADC3_IN15: now also J7.10
- net ADC3_IN4: now also J7.11
- net ADC3_IN5: now also J7.12
- net ADC3_IN6: now also J7.13
- net ADC3_IN7: now also J7.14
- net ADC3_IN8: now also J7.15, J7.8
- net CAN1_RX: now also J5.2
- net CAN1_TX: now also J5.1
- net DAC1: now also J4.20
- net GND: now also C31.2, U$15.P$1; no longer J3.20, J4.20, J5.20, J6.20, J7.20
- net I2C2_SDA: now also J3.18
- net I2C2_SMBA: now also J3.20
- net I2C3_SCL: now also J6.2; no longer R3.1, U$1G$6.PF1
- net I2C3_SDA: now also J6.1
- net I2C3_SMBA: now also J6.3
- net PA15: now also J3.5
- net PB14: now also J3.7
- net PB4: now also J3.6
- net PC15: now also J3.8
- net PD0: now also J3.9
- net PD1: now also J3.10
- net PD10: now also J4.3
- net PD11: now also J4.4
- net PD12: now also J4.5
- net PD13: now also J4.6
- net PD14: now also J4.7
- net PD15: now also J4.8
- net PD3: now also J3.11
- net PD4: now also J3.12
- net PD5: now also J3.13
- net PD6: now also J3.14
- net PD7: now also J3.15
- net PD8: now also J3.16
- net PD9: now also J3.17
- net PE0: now also J4.9
- net PE1: now also J4.10
- net PE10: now also J4.19
- net PE11: now also J5.3
- net PE12: now also J5.4
- net PE13: now also J5.5
- net PE14: now also J5.6
- net PE15: now also J5.7
- net PE2: now also J4.11
- net PE3: now also J4.12
- net PE4: now also J4.13
- net PE5: now also J4.14
- net PE6: now also J4.15
- net PE7: now also J4.16
- net PE8: now also J4.17
- net PE9: now also J4.18
- net PF11: now also J5.8
- net PF12: now also J5.9
- net PF13: now also J5.10
- net PF14: now also J5.11
- net PF15: now also J5.12
- net PG0: now also J5.13
- net PG1: now also J5.14
- net PG10: now also J6.6
- net PG11: now also J6.7
- net PG12: now also J6.8
- net PG13: now also J6.9
- net PG14: now also J6.10
- net PG15: now also J6.11
- net PG2: now also J5.15
- net PG3: now also J5.16
- net PG4: now also J5.17
- net PG5: now also J5.18
- net PG6: now also J5.19
- net PG7: now also J5.20
- net PG8: now also J6.4
- net PG9: now also J6.5
- net PH10: now also J6.16
- net PH11: now also J6.17
- net PH12: now also J6.18
- net PH14: now also J6.19
- net PH15: now also J6.20
- net PH2: now also J6.12
- net PH3: now also J6.13
- net PH5: now also J6.14
- net PH6: now also J6.15
- net PI4: now also J7.16
- net PI5: now also J7.17
- net PI6: now also J7.18
- net PI7: now also J7.19
- net PI8: now also J7.20
- net SPI2_MISO: now also J3.3
- net SPI2_MOSI: now also J3.4
- net SPI2_NSS: now also J3.1
- net SPI2_SCK: now also J3.2
- net UART4_RX: now also J4.2
- net UART4_TX: now also J4.1
Other:
- note added: "*Finish SWD connector *ULPI CPEN *Find 1.8V supply *BOOT0/BOOT1 conector"
- note added: "TO DO:"
- moved on the sheet: J3, J4, J5, J6, J7

Commit message: Added RGB led and resistors
Parts:
- added LED1: (no value), led-rgb-rohm:LED_RGB_COMMON_ANODE-1.6X1.26
- added R12, R13, R14: (no value), rcl_custom:R-US_0603-C
- U$1: PB8 SDIO_D4 -> GPIO; PB9 SDIO_D5 -> GPIO; PC6 SDIO_D6 -> GPIO; PC7 SDIO_D7 -> GPIO
Connections:
- net SDIO_D7 renamed PC6
- removed net SDIO_D4: U$1G$2.PB8
- removed net SDIO_D5: U$1G$2.PB9
- removed net SDIO_D6: U$1G$3.PC6
- new net B_LED: R14.1, U$1G$3.PC6
- new net G_LED: R13.1, U$1G$2.PB9
- new net N$16: LED1.RK, R12.2
- new net N$17: LED1.GK, R13.2
- new net N$18: LED1.BK, R14.2
- new net R_LED: R12.1, U$1G$2.PB8
- net +3.3VDD: now also LED1.COMMON_ANODE
Other:
- moved on the sheet: R6, R7

Commit message: library update/maintinence and added pullup and pulldown resisters
Parts:
- added C32: 1uF, 10V, rcl_custom:C-EU0603-C
- added R15: 820, rcl_custom:R-US_0603-C
- added R16, R17, R18: 10k, rcl_custom:R-US_0603-C
- J2: value SWD_CONNECTOR -> SWD; device SWD_CONNECTOR:SWD_CONNECTOR -> SWD_CONNECTOR:SWD
- R12: value (none) -> 68
- R13, R14: value (none) -> 5.1
Connections:
- removed net N$13: C31.1, U$15.P$2, U$1G$11.NRST
- new net NRST: C31.1, J2.RESET, R18.1, U$15.P$2, U$1G$11.NRST
- net +3.3VDD: now also R16.2, R17.2, R18.2
- net GND: now also C28.2, C32.2, R1.2, U1.GND
- net N$12: now also R15.2, U1.VBUS; no longer C28.2, R1.2, U1.GND
- net N$2: now also C32.1, R15.1; no longer U1.VBUS
- net SWDIO: now also R17.1
- net SWO: now also R16.1
Other:
- note added: "*See figure 8.1 in USB3318 datasheet"
- moved on the sheet: C28, C29, LED1, R12, R13, R14, R6, R7, U$3

Commit message: Added super cap and circuitry
Parts:
- added C33: EDLC, DCK3R3:EDLC
- added D3: CDBU0530, CBDU0530:CDBU0530
- added R19: (no value), rcl_custom:R-US_0603-C
Connections:
- new net N$13: D3.A, R19.1
- new net N$15: C33.P$1, D3.C, U$1G$11.VBATT
- net +3.3VDD: now also R19.2
- net GND: now also C33.P$2
Changed lines of the file:
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@@
 <part name="R17" library="rcl_custom" deviceset="R-US_" device="0603-C" value="10k"/>
 <part name="R18" library="rcl_custom" deviceset="R-US_" device="0603-C" value="10k"/>
+<part name="C33" library="DCK3R3" deviceset="EDLC" device=""/>
+<part name="D3" library="CBDU0530" deviceset="CDBU0530" device=""/>
+<part name="R19" library="rcl_custom" deviceset="R-US_" device="0603-C"/>
+<part name="U$17" library="3_3VDDsupply" deviceset="+3.3VDD" device=""/>
 </parts>
 <sheets>
@@
 <instance part="U$15" gate="G$1" x="146.05" y="93.98"/>
 <instance part="C31" gate="CE" x="147.32" y="88.9" smashed="yes" rot="R270">
-<attribute name="NAME" x="148.336" y="85.979" size="1.778" layer="95" rot="R180"/>
-<attribute name="VALUE" x="141.224" y="81.661" size="1.778" layer="96"/>
+<attribute name="NAME" x="144.526" y="88.519" size="1.778" layer="95" rot="R180"/>
+<attribute name="VALUE" x="163.576" y="88.519" size="1.778" layer="96" rot="R180"/>
 </instance>
 <instance part="GND9" gate="1" x="130.81" y="83.82"/>
+<instance part="C33" gate="G$1" x="123.19" y="99.06"/>
+<instance part="D3" gate="G$1" x="110.49" y="104.14"/>
+<instance part="R19" gate="R" x="102.87" y="115.57" rot="R90"/>
+<instance part="U$17" gate="G$1" x="102.87" y="127"/>
 </instances>
 <busses>
@@
 <junction x="130.81" y="88.9"/>
 <pinref part="GND9" gate="1" pin="GND"/>
+<pinref part="C33" gate="G$1" pin="P$2"/>
+<wire x1="123.19" y1="96.52" x2="123.19" y2="91.44" width="0.1524" layer="91"/>
+<wire x1="123.19" y1="91.44" x2="125.73" y2="88.9" width="0.1524" layer="91"/>
+<wire x1="125.73" y1="88.9" x2="130.81" y2="88.9" width="0.1524" layer="91"/>
 </segment>
 </net>
@@
 <pinref part="U$8" gate="G$1" pin="+3.3VDD"/>
 </segment>
+<segment>
+<pinref part="R19" gate="R" pin="2"/>
+<pinref part="U$17" gate="G$1" pin="+3.3VDD"/>
+<wire x1="102.87" y1="120.65" x2="102.87" y2="124.46" width="0.1524" layer="91"/>
+</segment>
 </net>
 <net name="FS_ID" class="0">
@@
 </segment>
 </net>
+<net name="N$15" class="0">
+<segment>
+<pinref part="C33" gate="G$1" pin="P$1"/>
+<wire x1="123.19" y1="101.6" x2="123.19" y2="104.14" width="0.1524" layer="91"/>
+<wire x1="123.19" y1="104.14" x2="190.5" y2="104.14" width="0.1524" layer="91"/>
+<wire x1="190.5" y1="104.14" x2="195.58" y2="99.06" width="0.1524" layer="91"/>
+<pinref part="U$1" gate="G$11" pin="VBATT"/>
+<wire x1="195.58" y1="99.06" x2="223.52" y2="99.06" width="0.1524" layer="91"/>
+<pinref part="D3" gate="G$1" pin="C"/>
+<wire x1="123.19" y1="104.14" x2="113.03" y2="104.14" width="0.1524" layer="91"/>
+<junction x="123.19" y="104.14"/>
+</segment>
+</net>
+<net name="N$13" class="0">
+<segment>
+<pinref part="D3" gate="G$1" pin="A"/>
+<wire x1="107.95" y1="104.14" x2="105.41" y2="104.14" width="0.1524" layer="91"/>
+<wire x1="105.41" y1="104.14" x2="102.87" y2="106.68" width="0.1524" layer="91"/>
+<wire x1="102.87" y1="106.68" x2="102.87" y2="110.49" width="0.1524" layer="91"/>
+<pinref part="R19" gate="R" pin="1"/>
+</segment>
+</net>
 </nets>
 </sheet>
@@
 </segment>
 </net>
+<net name="PC6" class="0">
+<segment>
+<wire x1="-118.11" y1="-195.58" x2="-115.57" y2="-198.12" width="0.1524" layer="91"/>
+<wire x1="-115.57" y1="-198.12" x2="-101.6" y2="-198.12" width="0.1524" layer="91"/>
+<label x="-107.95" y="-198.12" size="1.778" layer="95"/>
+</segment>
+</net>

Commit message: Added 16Mhz clock to schematic
Parts:
- added C34, C35: 4.4nF, rcl_custom:C-EU0603-C
- added R20: 2.26k, rcl_custom:R-US_0603-C
- added U$18: NX3225SA, NX3225SA:NX3225SA
Connections:
- new net N$19: C35.1, U$18.P$2, U$1G$8.PH0
- new net N$20: R20.1, U$1G$8.PH1
- new net N$21: C34.1, R20.2, U$18.P$1
- net GND: now also C34.2, C35.2
Changed lines of the file:
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@@
 <setting verticaltext="up"/>
 </settings>
-<grid distance="0.05" unitdist="inch" unit="inch" style="lines" multiple="1" display="yes" altdistance="0.01" altunitdist="inch" altunit="inch"/>
+<grid distance="0.1" unitdist="inch" unit="inch" style="lines" multiple="1" display="yes" altdistance="0.01" altunitdist="inch" altunit="inch"/>
 <layers>
 <layer number="1" name="Top" color="4" fill="1" visible="no" active="no"/>
@@
 <part name="R19" library="rcl_custom" deviceset="R-US_" device="0603-C"/>
 <part name="U$17" library="3_3VDDsupply" deviceset="+3.3VDD" device=""/>
+<part name="U$18" library="NX3225SA" deviceset="NX3225SA" device=""/>
+<part name="R20" library="rcl_custom" deviceset="R-US_" device="0603-C" value="2.26k"/>
+<part name="C34" library="rcl_custom" deviceset="C-EU" device="0603-C" value="4.4nF"/>
+<part name="C35" library="rcl_custom" deviceset="C-EU" device="0603-C" value="4.4nF"/>
+<part name="GND13" library="GROUND" deviceset="GND" device=""/>
 </parts>
 <sheets>
@@
 <instance part="FRAME2" gate="G$1" x="-194.31" y="-200.66"/>
 <instance part="FRAME2" gate="G$2" x="257.81" y="-200.66"/>
+<instance part="U$18" gate="G$1" x="53.34" y="50.8"/>
+<instance part="R20" gate="R" x="40.64" y="45.72" rot="R90"/>
+<instance part="C34" gate="CE" x="45.72" y="43.18"/>
+<instance part="C35" gate="CE" x="60.96" y="43.18"/>
+<instance part="GND13" gate="1" x="53.34" y="33.02"/>
 </instances>
 <busses>
@@
 </segment>
 </net>
+<net name="N$19" class="0">
+<segment>
+<pinref part="U$1" gate="G$8" pin="PH0"/>
+<wire x1="-66.04" y1="35.56" x2="35.56" y2="35.56" width="0.1524" layer="91"/>
+<wire x1="35.56" y1="35.56" x2="35.56" y2="60.96" width="0.1524" layer="91"/>
+<wire x1="35.56" y1="60.96" x2="60.96" y2="60.96" width="0.1524" layer="91"/>
+<pinref part="U$18" gate="G$1" pin="P$2"/>
+<wire x1="60.96" y1="60.96" x2="60.96" y2="50.8" width="0.1524" layer="91"/>
+<wire x1="60.96" y1="50.8" x2="60.96" y2="45.72" width="0.1524" layer="91"/>
+<pinref part="C35" gate="CE" pin="1"/>
+</segment>
+</net>
+<net name="N$20" class="0">
+<segment>
+<pinref part="U$1" gate="G$8" pin="PH1"/>
+<wire x1="-66.04" y1="30.48" x2="40.64" y2="30.48" width="0.1524" layer="91"/>
+<pinref part="R20" gate="R" pin="1"/>
+<wire x1="40.64" y1="30.48" x2="40.64" y2="40.64" width="0.1524" layer="91"/>
+</segment>
+</net>
+<net name="N$21" class="0">
+<segment>
+<pinref part="R20" gate="R" pin="2"/>
+<pinref part="U$18" gate="G$1" pin="P$1"/>
+<wire x1="40.64" y1="50.8" x2="45.72" y2="50.8" width="0.1524" layer="91"/>
+<wire x1="45.72" y1="50.8" x2="45.72" y2="45.72" width="0.1524" layer="91"/>
+<pinref part="C34" gate="CE" pin="1"/>
+</segment>
+</net>
+<net name="GND" class="0">
+<segment>
+<pinref part="C34" gate="CE" pin="2"/>
+<pinref part="C35" gate="CE" pin="2"/>
+<wire x1="45.72" y1="38.1" x2="53.34" y2="38.1" width="0.1524" layer="91"/>
+<pinref part="GND13" gate="1" pin="GND"/>
+<wire x1="53.34" y1="38.1" x2="60.96" y2="38.1" width="0.1524" layer="91"/>
+<wire x1="53.34" y1="38.1" x2="53.34" y2="35.56" width="0.1524" layer="91"/>
+</segment>
+</net>

Commit message: Edited device prefix
Parts:
- removed U$18: NX3225SA, NX3225SA:NX3225SA
- added X2: NX3225SA, NX3225SA:NX3225SA
Connections:
- removed net N$19: C35.1, U$18.P$2, U$1G$8.PH0
- new net N$23: C35.1, U$1G$8.PH0, X2.P$2
- net N$21: now also X2.P$1; no longer U$18.P$1
Other:
- moved on the sheet: C34, C35, R20

Commit message: Added notes and changes from rough draft review
Parts:
- R19: value (none) -> 1k
Connections:
- net GND: now also J2.GND_DETECT
Other:
- note added: "* MCO1 is clock out from MCU maybe add a net out to a test point or male pin"
- note added: "add diode and connect to 5v Vbus on supply"
- note removed: "* MCO1 is clock out from MCU"
Changed lines of the file:
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@@
 <setting verticaltext="up"/>
 </settings>
-<grid distance="0.1" unitdist="inch" unit="inch" style="lines" multiple="1" display="yes" altdistance="0.01" altunitdist="inch" altunit="inch"/>
+<grid distance="0.05" unitdist="inch" unit="inch" style="lines" multiple="1" display="yes" altdistance="0.01" altunitdist="inch" altunit="inch"/>
 <layers>
 <layer number="1" name="Top" color="4" fill="1" visible="no" active="no"/>
@@
 <part name="C33" library="DCK3R3" deviceset="EDLC" device=""/>
 <part name="D3" library="CBDU0530" deviceset="CDBU0530" device=""/>
-<part name="R19" library="rcl_custom" deviceset="R-US_" device="0603-C"/>
+<part name="R19" library="rcl_custom" deviceset="R-US_" device="0603-C" value="1k"/>
 <part name="U$17" library="3_3VDDsupply" deviceset="+3.3VDD" device=""/>
 <part name="R20" library="rcl_custom" deviceset="R-US_" device="0603-C" value="2.26k"/>
@@
 <part name="GND13" library="GROUND" deviceset="GND" device=""/>
 <part name="X2" library="NX3225SA" deviceset="NX3225SA" device=""/>
+<part name="GND14" library="GROUND" deviceset="GND" device=""/>
 </parts>
 <sheets>
@@
 <plain>
 <text x="-125.73" y="86.36" size="3.81" layer="94">NOTES</text>
-<text x="-123.19" y="82.55" size="1.9304" layer="97">* MCO1 is clock out from MCU</text>
+<text x="-133.35" y="77.47" size="1.9304" layer="97">* MCO1 is clock out from MCU
+maybe add a net out to a test point or male pin
+</text>
 <text x="-123.19" y="76.2" size="1.778" layer="97">TO DO:</text>
 <text x="-120.65" y="64.77" size="1.778" layer="97">*Finish SWD connector
@@
 *BOOT0/BOOT1 conector</text>
 <text x="256.54" y="81.28" size="1.778" layer="97">*See figure 8.1 in USB3318 datasheet</text>
+<text x="299.72" y="96.52" size="1.778" layer="97">add diode and connect to 5v Vbus on supply</text>
 </plain>
 <instances>
@@
 <pinref part="J2" gate="G$1" pin="GND@1"/>
 <pinref part="J2" gate="G$1" pin="GND"/>
-<wire x1="149.86" y1="55.88" x2="149.86" y2="43.18" width="0.1524" layer="91"/>
+<wire x1="149.86" y1="55.88" x2="149.86" y2="50.8" width="0.1524" layer="91"/>
+<wire x1="149.86" y1="50.8" x2="149.86" y2="43.18" width="0.1524" layer="91"/>
 <wire x1="143.51" y1="58.42" x2="147.32" y2="58.42" width="0.1524" layer="91"/>
 <wire x1="147.32" y1="58.42" x2="149.86" y2="55.88" width="0.1524" layer="91"/>
 <junction x="149.86" y="55.88"/>
+<pinref part="J2" gate="G$1" pin="GND_DETECT"/>
+<wire x1="143.51" y1="50.8" x2="149.86" y2="50.8" width="0.1524" layer="91"/>
+<junction x="149.86" y="50.8"/>
 </segment>
 </net>
@@
 <segment>
 <pinref part="U$3" gate="G$1" pin="VCC"/>
-<wire x1="292.1" y1="73.66" x2="304.8" y2="73.66" width="0.1524" layer="91"/>
+<wire x1="292.1" y1="73.66" x2="297.18" y2="73.66" width="0.1524" layer="91"/>
+<wire x1="297.18" y1="73.66" x2="304.8" y2="73.66" width="0.1524" layer="91"/>
 <wire x1="292.1" y1="73.66" x2="292.1" y2="60.96" width="0.1524" layer="91"/>
 <pinref part="C32" gate="CE" pin="1"/>
@@
 <wire x1="274.32" y1="73.66" x2="292.1" y2="73.66" width="0.1524" layer="91"/>
 <junction x="292.1" y="73.66"/>
+<wire x1="297.18" y1="73.66" x2="297.18" y2="96.52" width="0.1524" layer="91"/>
+<junction x="297.18" y="73.66"/>
 </segment>
 </net>
@@
 <instance part="R19" gate="R" x="102.87" y="115.57" rot="R90"/>
 <instance part="U$17" gate="G$1" x="102.87" y="127"/>
+<instance part="GND14" gate="1" x="123.19" y="88.9"/>
 </instances>
 <busses>
@@
 <junction x="130.81" y="88.9"/>
 <pinref part="GND9" gate="1" pin="GND"/>
+</segment>
+<segment>
 <pinref part="C33" gate="G$1" pin="P$2"/>
 <wire x1="123.19" y1="96.52" x2="123.19" y2="91.44" width="0.1524" layer="91"/>
-<wire x1="123.19" y1="91.44" x2="125.73" y2="88.9" width="0.1524" layer="91"/>
-<wire x1="125.73" y1="88.9" x2="130.81" y2="88.9" width="0.1524" layer="91"/>
-</segment>
-</net>
+<pinref part="GND14" gate="1" pin="GND"/>
+</segment>
+</net>

Commit message: Added SD detect, fixed some gpio stuff, added some other labels
Parts:
- removed R17, R18: 10k, rcl_custom:R-US_0603-C
- removed R20: 2.26k, rcl_custom:R-US_0603-C
- added C36: 0.1uF, 10V, rcl_custom:C-EU0603-C
- added D4: CDBU0530, CBDU0530:CDBU0530
- U$1: PC7 GPIO -> SD_DETECT
Connections:
- removed net N$21: C34.1, R20.2, X2.P$1
- removed net N$8: C1.1, C3.1, D1.C, D2.C, U2.EN, U2.IN, U3.CE/MODE, U3.VIN
- removed net PC6: U$1G$3.PC7
- new net MCO1: U$1G$1.PA8
- new net SD_DETECT: U$13CD.0, U$1G$3.PC7
- new net VCC: C1.1, C3.1, D1.C, D2.C, D4.C, U2.EN, U2.IN, U3.CE/MODE, U3.VIN
- net +3.3VDD: no longer R17.2, R18.2
- net GND: now also C36.1, C36.2, U$13CD.1
- net N$2: now also D4.A
- net N$20: now also C34.1, X2.P$1; no longer R20.1
- net NRST: now also R16.1; no longer R18.1
- net SWDIO: no longer R17.1
- net SWO: no longer R16.1
Other:
- note added: "*Find 1.8V supply *BOOT0/BOOT1 conector"
- note removed: "*Finish SWD connector *ULPI CPEN *Find 1.8V supply *BOOT0/BOOT1 conector"
- note removed: "add diode and connect to 5v Vbus on supply"
- moved on the sheet: C32, U$3
