File: current_amplifier/imon.sch (EAGLE design)
At the start: 70 parts, among them U2 OPAMP_DUALFAN4852, U4 AD8418, U5 MCP1501", U6 LTC2312-12

Commit message: added note about adding reverse polarity protection
Parts:
- added R9: 0, rcl_custom:R-US_0402-B
- added TP3: PAD+VIA_0.3302MM, dock_v2:PAD+VIA_0.3302MM
- R7, R8: value 10 -> 0
Connections:
- new net OPAMP_IN+: R9.1, TP3.TP, U2G1.+IN, U2G2.+IN
- net GND: no longer U2G1.+IN, U2G2.+IN
- net VREF_FILTERED: now also R9.2
Other:
- note added: "Add part number for a terminal block"
- note added: "Add reverse polarity protection. Absolutely necessary because these boards get daisy chained together in big arrays and then one short circuit would toast all 8 of our boards."
- note added: "Change order of VSHUNT_20X_OUT and VSHUNT_FILTERED so that the pin closest to the DM/DP raw signal is the least processed."
- note added: "Low Pass 4th Ord. Bessel Filter"
- note added: "Make an intelligent connection of the + input terminals of opamps bearing in mind the different configurations of VREF1/VREF2 of the AD8418. The stages are inverting so it is probably necessary for OPAMPIN+ to be either VREF or some other voltage that is in the middle of the range."
- note removed: "Low Pass 4th or. Bessel Filter"
- moved on the sheet: C1, C105, C14, C15, C7, J1, R12, R18, R19, R5, R6, TP1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
