File: current_amplifier/imon.brd (EAGLE design)
At the start: 81 x 16 mm, 70 parts, among them U2 OPAMP_DUALFAN4852, U4 AD8418, U5 MCP1501", U6 LTC2312-12

Commit message: some small changes
Parts:
- added R9: 0, rcl_custom:.0402-B
- added TP3: PAD+VIA_0.3302MM, dock_v2:PAD+VIA_0.3302MM
- R7, R8: value 10 -> 0
Connections:
- new net OPAMP_IN+: R9.1, TP3.TP, U2.3, U2.5
- net GND: no longer U2.3, U2.5
- net VREF_FILTERED: now also R9.2
Routing:
- net OPAMP_IN+: track 0.00 -> 1.71 mm
Other:
- outline, holes or cut-outs redrawn
- board text added: "Add pinout notation to top of board (at least V5D and GND)"
- board text added: "Add tplace rectangle for annotation"
- board text added: "Choose a terminal block, probably the black terminal block 3.5mm WM7877-ND"
